Commit message: update agv_pro_description/urdf/agv_pro.urdf

File: agv_pro_description/urdf/agv_pro.urdf (robot description, URDF)
Before this commit: robot AGV pro, 7 links, 6 joints
Links:
- removed link base_scan
- added link laser_link, mass 0; collision mesh filename=package://agv_pro_description/meshes/lidar.stl; visual mesh filename=package://agv_pro_description/meshes/lidar.stl
Joints:
- joint lidar_joint: child base_scan -> laser_link

Commit message: update agv_pro_description/

File: agv_pro_description/urdf/agv_pro.urdf (robot description, URDF)
Before this commit: robot AGV pro, 7 links, 6 joints
Links:
- link base_link: mass 17.2325340030774 -> 19.236
- link laser_link: mass 0 -> 0.049095; geometry collision mesh filename=package://agv_pro_description/meshes/laser_link.stl; visual mesh filename=package://agv_pro_description/meshes/laser_link.stl
- link left_front_wheel_link: mass 0.216591225420666 -> 0.3015; geometry collision mesh filename=package://agv_pro_description/meshes/wheel_lf_link.stl; visual mesh filename=package://agv_pro_description/meshes/wheel_lf_link.stl
- link left_rear_wheel_link: mass 0.21659122149267 -> 0.29613; geometry collision mesh filename=package://agv_pro_description/meshes/wheel_lb_link.stl; visual mesh filename=package://agv_pro_description/meshes/wheel_lb_link.stl
- link right_front_wheel_link: geometry collision mesh filename=package://agv_pro_description/meshes/wheel_rf_link.stl; visual mesh filename=package://agv_pro_description/meshes/wheel_rf_link.stl
- link right_rear_wheel_link: geometry collision mesh filename=package://agv_pro_description/meshes/wheel_rb_link.stl; visual mesh filename=package://agv_pro_description/meshes/wheel_rb_link.stl
Joints:
- removed joint Left_front_wheel_joint
- added joint left_front_wheel_joint: type continuous, parent base_link, child left_front_wheel_link, origin xyz=0.17128 0.1799 0.052 rpy=0 0 0, axis 0 1 0
- joint base_joint: origin xyz=0 0 0.010 rpy=0 0 0 -> xyz=0 0 0.020 rpy=0 0 0
- joint left_rear_wheel_joint: axis 0 0 0 -> 0 1 0; origin xyz=-0.1239 0.142 0.052 rpy=0 0 0 -> xyz=0.17128 -0.1799 0.052 rpy=0 0 0; type fixed -> continuous
- joint lidar_joint: origin xyz=0.22254 0 0.2339 rpy=0 0 0 -> xyz=0.17891 0 0.20928 rpy=0 0 0
- joint right_front_wheel_joint: axis 0 0 0 -> 0 1 0; origin xyz=0.2191 -0.142 0.052 rpy=0 0 0 -> xyz=-0.17181 0.1799 0.051884 rpy=0 0 0; type fixed -> continuous
- joint right_rear_wheel_joint: axis 0 0 0 -> 0 1 0; origin xyz=-0.1239 -0.142 0.052 rpy=0 0 0 -> xyz=-0.171806101587598 -0.179900399999999 0.0518836514526621 rpy=0 0 0; type fixed -> continuous

Commit message: add agvpro_display.rviz

File: agv_pro_description/urdf/agv_pro.urdf (robot description, URDF)
Before this commit: robot AGV pro, 7 links, 6 joints
Joints:
- joint lidar_joint: axis 0 0 0 -> (none)

Commit message: Add a namespace for multi-machine control

File: agv_pro_description/urdf/agv_pro.urdf (robot description, URDF)
Before this commit: robot AGV pro, 7 links, 6 joints
Links:
- removed link base_footprint
- removed link base_link
- removed link laser_link
- removed link left_front_wheel_link
- removed link left_rear_wheel_link
- removed link right_front_wheel_link
- removed link right_rear_wheel_link
- added link ${namespace}base_footprint
- added link ${namespace}base_link, mass 19.236; collision mesh filename=package://agv_pro_description/meshes/base_link.stl; visual mesh filename=package://agv_pro_description/meshes/base_link.stl
- added link ${namespace}laser_link, mass 0.049095; collision mesh filename=package://agv_pro_description/meshes/laser_link.stl; visual mesh filename=package://agv_pro_description/meshes/laser_link.stl
- added link ${namespace}left_front_wheel_link, mass 0.3015; collision mesh filename=package://agv_pro_description/meshes/wheel_lf_link.stl; visual mesh filename=package://agv_pro_description/meshes/wheel_lf_link.stl
- added link ${namespace}left_rear_wheel_link, mass 0.29613; collision mesh filename=package://agv_pro_description/meshes/wheel_lb_link.stl; visual mesh filename=package://agv_pro_description/meshes/wheel_lb_link.stl
- added link ${namespace}right_front_wheel_link, mass 0.21659122149244; collision mesh filename=package://agv_pro_description/meshes/wheel_rf_link.stl; visual mesh filename=package://agv_pro_description/meshes/wheel_rf_link.stl
- added link ${namespace}right_rear_wheel_link, mass 0.21659; collision mesh filename=package://agv_pro_description/meshes/wheel_rb_link.stl; visual mesh filename=package://agv_pro_description/meshes/wheel_rb_link.stl
Joints:
- removed joint base_joint
- removed joint left_front_wheel_joint
- removed joint left_rear_wheel_joint
- removed joint lidar_joint
- removed joint right_front_wheel_joint
- removed joint right_rear_wheel_joint
- added joint ${namespace}base_joint: type fixed, parent ${namespace}base_footprint, child ${namespace}base_link, origin xyz=0 0 0.020 rpy=0 0 0
- added joint ${namespace}left_front_wheel_joint: type continuous, parent ${namespace}base_link, child ${namespace}left_front_wheel_link, origin xyz=0.17128 0.1799 0.052 rpy=0 0 0, axis 0 1 0
- added joint ${namespace}left_rear_wheel_joint: type continuous, parent ${namespace}base_link, child ${namespace}left_rear_wheel_link, origin xyz=0.17128 -0.1799 0.052 rpy=0 0 0, axis 0 1 0
- added joint ${namespace}lidar_joint: type fixed, parent ${namespace}base_link, child ${namespace}laser_link, origin xyz=0.17891 0 0.20928 rpy=0 0 0
- added joint ${namespace}right_front_wheel_joint: type continuous, parent ${namespace}base_link, child ${namespace}right_front_wheel_link, origin xyz=-0.17181 0.1799 0.051884 rpy=0 0 0, axis 0 1 0
- added joint ${namespace}right_rear_wheel_joint: type continuous, parent ${namespace}base_link, child ${namespace}right_rear_wheel_link, origin xyz=-0.171806101587598 -0.179900399999999 0.0518836514526621 rpy=0 0 0, axis 0 1 0
